File: Leonardo/Leonardo.sch (KiCad schematic (older format))
At the start: 49 parts, among them J1 Conn_01x08_Female, J2 Conn_01x06_Female, J3 Conn_01x10_Female, J4 Conn_01x08_Female, J5 Conn_02x03_Odd_Even, J6 USB_Micro, J7 Barrel_Jack, Q1 FDN340P, SW1 TL3342, U1 LMV358IDGKR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

Commit message: Initial layout
Parts:
- D5: footprint Diodes_SMD:D_0805 -> Diodes_SMD:D_SMB
- J1: value Conn_01x08_Female -> Power
- J2: value Conn_01x06_Female -> Analog
- J3: value Conn_01x10_Female -> Digital_2
- J4: value Conn_01x08_Female -> Digital_1
- J5: value Conn_02x03_Odd_Even -> ISP
Connections:
- net xD-: now reaches J6.2 (D-), R10.2, RV1.1
- net xD+: now reaches J6.3 (D+), R9.2, RV2.1
Changed lines of the file:
@@
 F 0 "D5" H 9100 5200 50  0000 C CNN
 F 1 "M7" H 9100 5000 50  0000 C CNN
-F 2 "Diodes_SMD:D_0805" H 9100 5100 50  0001 C CNN
+F 2 "Diodes_SMD:D_SMB" H 9100 5100 50  0001 C CNN
 F 3 "" H 9100 5100 50  0001 C CNN
 	1    9100 5100
@@
 P 4600 7250
 F 0 "J2" H 4600 7550 50  0000 C CNN
-F 1 "Conn_01x06_Female" H 4600 6850 50  0000 C CNN
+F 1 "Analog" H 4600 6850 50  0000 C CNN
 F 2 "Socket_Strips:Socket_Strip_Straight_1x06_Pitch2.54mm" H 4600 7250 50  0001 C CNN
 F 3 "" H 4600 7250 50  0001 C CNN
@@
 P 4600 6100
 F 0 "J1" H 4600 6500 50  0000 C CNN
-F 1 "Conn_01x08_Female" H 4600 5600 50  0000 C CNN
+F 1 "Power" H 4600 5600 50  0000 C CNN
 F 2 "Socket_Strips:Socket_Strip_Straight_1x08_Pitch2.54mm" H 4600 6100 50  0001 C CNN
 F 3 "" H 4600 6100 50  0001 C CNN
@@
 P 5400 7150
 F 0 "J4" H 5400 7550 50  0000 C CNN
-F 1 "Conn_01x08_Female" H 5400 6650 50  0000 C CNN
+F 1 "Digital_1" H 5400 6650 50  0000 C CNN
 F 2 "Socket_Strips:Socket_Strip_Straight_1x08_Pitch2.54mm" H 5400 7150 50  0001 C CNN
 F 3 "" H 5400 7150 50  0001 C CNN
@@
 P 5400 6000
 F 0 "J3" H 5400 6500 50  0000 C CNN
-F 1 "Conn_01x10_Female" H 5400 5400 50  0000 C CNN
+F 1 "Digital_2" H 5400 5400 50  0000 C CNN
 F 2 "Socket_Strips:Socket_Strip_Straight_1x10_Pitch2.54mm" H 5400 6000 50  0001 C CNN
 F 3 "" H 5400 6000 50  0001 C CNN
@@
 P 6700 6100
 F 0 "J5" H 6750 6300 50  0000 C CNN
-F 1 "Conn_02x03_Odd_Even" H 6750 5900 50  0000 C CNN
+F 1 "ISP" H 6750 5900 50  0000 C CNN
 F 2 "Pin_Headers:Pin_Header_Straight_2x03_Pitch2.54mm" H 6700 6100 50  0001 C CNN
 F 3 "" H 6700 6100 50  0001 C CNN
@@
 Wire Wire Line
 	8600 3200 8400 3200
+Text Label 8500 3000 0    60   ~ 0
+xD+
+Text Label 8500 3100 0    60   ~ 0
+xD-
 $EndSCHEMATC

Commit message: Tidy up a few things
Parts:
- F1: footprint Fuse_Holders_and_Fuses:Fuse_SMD1206_Reflow -> MF-MSMF050-2..:FUSC4632X85N
Changed lines of the file:
@@
 F 0 "F1" V 9030 2800 50  0000 C CNN
 F 1 "MF-MSMF050-2 500mA" V 8875 2800 50  0000 C CNN
-F 2 "Fuse_Holders_and_Fuses:Fuse_SMD1206_Reflow" V 8880 2800 50  0001 C CNN
+F 2 "MF-MSMF050-2..:FUSC4632X85N" V 8880 2800 50  0001 C CNN
 F 3 "" H 8950 2800 50  0001 C CNN
 	1    8950 2800
